File: ee/integrated/blackpants.kicad_sch (KiCad schematic)
At the start: 28 parts, among them J1 Conn_01x08, J2 Conn_01x10, J3 Conn_ARM_SWD_TagConnect_TC203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, SW1 SW_Push, U1 STM32F042C6Ux, U11 TPSGM7227YUWQ10G

Commit message: Split the project and moved some things around.
Parts:
- removed J1: Conn_01x08, Connector_Harwin:Harwin_M20-89008xx_1x08_P2.54mm_Horizontal, symbol Connector_Generic:Conn_01x08
- removed J2: Conn_01x10, Connector_Harwin:Harwin_M20-89010xx_1x10_P2.54mm_Horizontal, symbol Connector_Generic:Conn_01x10
- removed JP2, JP3: SolderJumper_2_Bridged, Jumper:SolderJumper-2_P1.3mm_Bridged_Pad1.0x1.5mm, symbol Jumper:SolderJumper_2_Bridged
Other:
- added sheet Hardware (hardware.kicad_sch)
- note removed: "1"
- note removed: "2"
- note removed: "3"
- note removed: "4"
- note removed: "5"
- note removed: "6"
- note removed: "7"
- note removed: "8"
- note removed: "9 10 11 12 13 14 15 16"
