File: ee/integrated/dsi_bridge.kicad_sch (KiCad schematic)
At the start: 17 parts, among them J11 Conn_01x20_MountingPin, J12 Conn_01x20_MountingPin, U15 AP3032

Commit message: Split the project and moved some things around.
Parts:
- removed J11: Conn_01x20_MountingPin, Connector_FFC-FPC:Amphenol_F32Q-1A7x1-11020_1x20-1MP_P0.5mm_Horizontal, symbol Connector_Generic_MountingPin:Conn_01x20_MountingPin
- removed J12: Conn_01x20_MountingPin, Connector_FFC-FPC:Hirose_FH12-20S-0.5SH_1x20-1MP_P0.50mm_Horizontal, symbol Connector_Generic_MountingPin:Conn_01x20_MountingPin
Connections:
- no-connect marks 6 -> 0
