File: ee/integrated/keyboard.kicad_sch (KiCad schematic)
At the start: 10 parts, among them SW11 SW_Push, SW12 SW_Push, SW13 SW_Push, SW14 SW_Push, SW15 SW_Push, SW16 SW_Push, SW17 SW_Push, SW18 SW_Push, SW19 SW_Push

Commit message: Split the project and moved some things around.
Parts:
- U14: value ~ -> (none)
