File: ee/integrated/usb.kicad_sch (KiCad schematic)
At the start: 43 parts, among them J10 Conn_01x01_Pin, J4 USB_A, J5 USB_A, J6 Conn_01x01_Pin, J7 Conn_01x01_Pin, J9 Conn_01x01_Pin, U3 USB2514B_Bi, U4 MIC2026-1xM, U5 USBLC6-2SC6, U6 USBLC6-2SC6, U8 USBLC6-2SC6, Y1 24Mhz

Commit message: Split the project and moved some things around.
Parts:
- removed J10, J6, J7, J9: Conn_01x01_Pin, blackpants:1871059-1, symbol Connector:Conn_01x01_Pin
- removed R24, R25: 100K, Resistor_SMD:R_0402_1005Metric, symbol Device:R_Small
- removed U8: USBLC6-2SC6, Package_TO_SOT_SMD:SOT-23-6, symbol Power_Protection:USBLC6-2SC6
